File: LuffyBadge2019_BSides.kicad_pcb (KiCad board)
At the start: 2 copper layers, 100 x 100.2 mm, 14 parts, among them J1 Conn_02x03_Odd_Even, SW1 SW_DIP_x01, U1 ATtiny13A-PU

Commit message: Fix vcc path on right leg
Routing:
- net VCC: track 69.3 -> 77.4 mm, vias 1 -> 3
Changed lines of the file:
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@@
     (thickness 1.6)
     (drawings 9936)
-    (tracks 133)
+    (tracks 144)
     (zones 0)
     (modules 14)
@@
     (37 F.SilkS user)
     (38 B.Mask user)
-    (39 F.Mask user hide)
+    (39 F.Mask user)
     (40 Dwgs.User user)
     (41 Cmts.User user)
@@
   (segment (start 147.2 133.2) (end 148.385 132.015) (width 0.25) (layer F.Cu) (net 10))
   (segment (start 143 129) (end 147.2 133.2) (width 0.25) (layer F.Cu) (net 10))
-  (segment (start 131.925 129) (end 143 129) (width 0.25) (layer F.Cu) (net 10))
-  (segment (start 128.499999 132.425001) (end 131.925 129) (width 0.25) (layer F.Cu) (net 10))
-  (segment (start 126.19 133.275) (end 127.039999 132.425001) (width 0.25) (layer F.Cu) (net 10))
-  (segment (start 127.039999 132.425001) (end 128.499999 132.425001) (width 0.25) (layer F.Cu) (net 10))
   (segment (start 171.775 136.57) (end 173.255 138.05) (width 0.25) (layer B.Cu) (net 10))
   (segment (start 171.775 133.375) (end 171.775 136.57) (width 0.25) (layer B.Cu) (net 10))
+  (segment (start 127.039999 134.124999) (end 130.949999 134.124999) (width 0.25) (layer F.Cu) (net 10))
+  (segment (start 126.19 133.275) (end 127.039999 134.124999) (width 0.25) (layer F.Cu) (net 10))
+  (segment (start 130.949999 134.124999) (end 131.775 134.95) (width 0.25) (layer F.Cu) (net 10))
+  (via (at 138.625 134.15) (size 0.8) (drill 0.4) (layers F.Cu B.Cu) (net 10))
+  (segment (start 131.775 134.95) (end 137.825 134.95) (width 0.25) (layer F.Cu) (net 10))
+  (segment (start 137.825 134.95) (end 138.625 134.15) (width 0.25) (layer F.Cu) (net 10))
+  (segment (start 138.625 133.584315) (end 137.775 132.734315) (width 0.25) (layer B.Cu) (net 10))
+  (segment (start 138.625 134.15) (end 138.625 133.584315) (width 0.25) (layer B.Cu) (net 10))
+  (segment (start 137.775 132.734315) (end 137.775 129.875) (width 0.25) (layer B.Cu) (net 10))
+  (via (at 136.475 128.575) (size 0.8) (drill 0.4) (layers F.Cu B.Cu) (net 10))
+  (segment (start 137.775 129.875) (end 136.475 128.575) (width 0.25) (layer B.Cu) (net 10))
+  (segment (start 137.040685 128.575) (end 137.115685 128.5) (width 0.25) (layer F.Cu) (net 10))
+  (segment (start 136.475 128.575) (end 137.040685 128.575) (width 0.25) (layer F.Cu) (net 10))
+  (segment (start 142.5 128.5) (end 143 129) (width 0.25) (layer F.Cu) (net 10))
+  (segment (start 137.115685 128.5) (end 142.5 128.5) (width 0.25) (layer F.Cu) (net 10))
   (segment (start 141.525 130.725) (end 142.815 132.015) (width 0.25) (layer F.Cu) (net 11))
   (via (at 136.05 131.3) (size 0.8) (drill 0.4) (layers F.Cu B.Cu) (net 11))
